File: panel_rp2354_20x20/panel_mcu.kicad_sch (KiCad schematic)
At the start: 32 parts, among them SW1 SW_Push, SW2 SW_Push, U1 APS6404L-3SQR, U2 RP2354B_80QFN, Y1 ABM8-272-T3

Commit message: Fixed part rotation issues.  Remove J2 J3 LCSC part as it was incorrect.
Parts:
- L1: FT Rotation Offset (none) -> 180
- U1: FT Rotation Offset (none) -> -90
Changed lines of the file:
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@@
+			)
+		)
+		(property "FT Rotation Offset" "-90"
+			(at 68.58 76.2 0)
+			(effects
+				(font
+					(size 1.27 1.27)
+				)
+				(hide yes)
 			)
 		)
@@
 			)
 		)
+		(property "FT Rotation Offset" "180"
+			(at 140.97 78.74 0)
+			(effects
+				(font
+					(size 1.27 1.27)
+				)
+				(hide yes)
+			)
+		)
