File: panel_rp2354_20x20/panel_usb_power.kicad_sch (KiCad schematic)
At the start: 4 parts, among them J1 Conn_01x04, U43 AP2112K-3.3

Commit message: Fixed part rotation issues.  Remove J2 J3 LCSC part as it was incorrect.
Parts:
- U43: FT Rotation Offset (none) -> 90
Changed lines of the file:
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@@
+			)
+		)
+		(property "FT Rotation Offset" "90"
+			(at 214.63 48.26 0)
+			(effects
+				(font
+					(size 1.27 1.27)
+				)
+				(hide yes)
 			)
 		)
