File: panel_rp2354_20x20_v0p1/drivers.kicad_sch (KiCad schematic)
At the start: 96 parts, among them U10 UCC27517, U11 UCC27517, U12 UCC27517, U13 UCC27517, U14 UCC27517, U15 UCC27517, U16 UCC27517, U17 UCC27517, U18 UCC27517, U19 UCC27517, U20 UCC27517, U21 UCC27517, U22 UCC27517, U23 UCC27517, U24 UCC27517, U25 UCC27517, U26 UCC27517, U27 UCC27517, U28 UCC27517, U29 UCC27517, U3 UCC27517, U30 UCC27517, U31 UCC27517, U32 UCC27517, U33 UCC27517, U34 UCC27517, U35 UCC27517, U36 UCC27517, U37 UCC27517, U38 UCC27517, U39 UCC27517, U4 UCC27517, U40 UCC27517, U41 UCC27517, U42 UCC27517, U5 UCC27517, U6 UCC27517, U7 UCC27517, U8 UCC27517, U9 UCC27517

Commit message: prepare v0.1.3
Other:
- company: (none) -> IORodeo for Reiserlab @ Janelia
- title: (none) -> G6 panel 45mm RP2354
Changed lines of the file:
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@@
 	(generator_version "9.0")
 	(paper "User" 457.2 457.2)
+	(title_block
+		(title "G6 panel 45mm RP2354")
+		(date "2025-11-25")
+		(rev "v0.1.3")
+		(company "IORodeo for Reiserlab @ Janelia")
+	)
 	(text "Column Drivers"
 		(exclude_from_sim no)
