File: panel_rp2354_20x20_v0p1/panel_mcu.kicad_sch (KiCad schematic)
At the start: 32 parts, among them SW1 SW_Push, SW2 SW_Push, U1 APS6404L-3SQR, U2 RP2354B_80QFN, Y1 ABM8-272-T3

Commit message: prepare v0.1.3
Other:
- company: (none) -> IORodeo for Reiserlab @ Janelia
- title: (none) -> G6 panel 45mm RP2354
Changed lines of the file:
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@@
 	(generator_version "9.0")
 	(paper "User" 406.4 279.4)
+	(title_block
+		(title "G6 panel 45mm RP2354")
+		(date "2025-11-25")
+		(rev "v0.1.3")
+		(company "IORodeo for Reiserlab @ Janelia")
+	)
 	(circle
 		(center 139.7 76.835)
