File: panel_rp2354_20x20_v0p1/panel_rp2354_20x20.kicad_pcb (KiCad board)
At the start: 6 copper layers, 45.4 x 45.4 mm, 556 parts, among them J1 Conn_01x04, J2 Conn_01x05, J3 Conn_01x05, J4 Conn_01x05, J5 Conn_01x05, SW1 SW_Push, SW2 SW_Push, U1 APS6404L-3SQR, U10 UCC27517, U11 UCC27517, U12 UCC27517, U13 UCC27517, U14 UCC27517, U15 UCC27517, U16 UCC27517, U17 UCC27517, U18 UCC27517, U19 UCC27517, U2 RP2354B_80QFN, U20 UCC27517, U21 UCC27517, U22 UCC27517, U23 UCC27517, U24 UCC27517, U25 UCC27517, U26 UCC27517, U27 UCC27517, U28 UCC27517, U29 UCC27517, U3 UCC27517, U30 UCC27517, U31 UCC27517, U32 UCC27517, U33 UCC27517, U34 UCC27517, U35 UCC27517, U36 UCC27517, U37 UCC27517, U38 UCC27517, U39 UCC27517, U4 UCC27517, U40 UCC27517, U41 UCC27517, U42 UCC27517, U43 AP2112K-3.3, U5 UCC27517, U6 UCC27517, U7 UCC27517, U8 UCC27517, U9 UCC27517, Y1 ABM8-272-T3

Commit message: prepare v0.1.3
Parts:
- R10, R14, R18, R22, R26: value 165 -> R_T1
- R11, R15, R19, R23, R27: value 165 -> R_T2
- R12, R16, R20, R24, R28: value 270 -> R_T3
- R13, R17, R21, R25, R9: value 270 -> R_T0
Other:
- board text added: "${ISSUE_DATE}"
- board text added: "${REVISION}"
- board text added: "${TITLE}"
- board text added: "BOTTOM"
- board text added: "TOP"
- board text added: "boot"
- board text added: "run"
- board text removed: "RP2354 V0.1R2"
