File: panel_rp2354_20x20_v0p1/panel_rp2354_20x20.kicad_sch (KiCad schematic)
At the start: 0 parts

Commit message: prepare v0.1.3
Other:
- company: (none) -> IORodeo for Reiserlab @ Janelia
- title: (none) -> G6 panel 45mm RP2354
Changed lines of the file:
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@@
 	(paper "USLetter")
 	(title_block
-		(date "9 may 2016")
+		(title "G6 panel 45mm RP2354")
+		(date "2025-11-25")
+		(rev "v0.1.3")
+		(company "IORodeo for Reiserlab @ Janelia")
 	)
 	(text "Column Pins"
