File: panel_rp2354_20x20_v0p1/panel_usb_power.kicad_sch (KiCad schematic)
At the start: 4 parts, among them J1 Conn_01x04, U43 AP2112K-3.3

Commit message: prepare v0.1.3
Other:
- company: (none) -> IORodeo for Reiserlab @ Janelia
- title: (none) -> G6 panel 45mm RP2354
Changed lines of the file:
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@@
 	(generator_version "9.0")
 	(paper "A4")
+	(title_block
+		(title "G6 panel 45mm RP2354")
+		(date "2025-11-25")
+		(rev "v0.1.3")
+		(company "IORodeo for Reiserlab @ Janelia")
+	)
 	(text "3.3V Regulator"
 		(exclude_from_sim no)
